Commit message: [modify] Modify pipette button travel

File: assets/pipette_good/pipette_good.urdf (robot description, URDF)
Before this commit: robot pipette_good, 2 links, 1 joints
Joints:
- joint PrismaticJoint: limit lower=-0.005 upper=0. effort=10000000. velocity=0. -> lower=-0.002 upper=0.00467 effort=10000000. velocity=0.
